File: Interfaces.kicad_sch (KiCad schematic)
At the start: 18 parts, among them J10 SPI1_Headers, J12 QSPI_Header, J13 USR_BTN_EN, J2 I2C1_Headers, J4 LPUART1_Headers, J5 GPIO_Headder, J6 SPI_QSPI_Jumper

Commit message: Update
Parts:
- added FPC1: FPC_0545481072, Personal_Project:FPC_0545481072, symbol Personal_Projects:FPC_0545481072
- added FPC4: FPC_0545482072, Personal_Project:FPC_0545482072, symbol Personal_Projects:FPC_0545482072
Connections:
- net GND: now also FPC1.1, FPC1.10, FPC1.11 (MP1), FPC1.12 (MP2), FPC1.3, FPC1.5, FPC1.6, FPC1.8, FPC4.1, FPC4.10, FPC4.11, FPC4.12, FPC4.14, FPC4.15, FPC4.17, FPC4.18, FPC4.20, FPC4.21 (MP1), FPC4.22 (MP2), FPC4.3, FPC4.4, FPC4.6, FPC4.7, FPC4.9
- new net QSPI_CLK: FPC4.2
- new net QSPI_CS0: FPC4.5
- new net QSPI_IO0: FPC4.8
- new net QSPI_IO1: FPC4.13
- new net QSPI_IO2: FPC4.16
- new net QSPI_IO3: FPC4.19
- new net SPI_CLK: FPC1.7
- new net SPI_CS: FPC1.9
- new net SPI_MISO: FPC1.4
- new net SPI_MOSI: FPC1.2

Commit message: Update
Parts:
- removed C5: 1uF, Capacitor_SMD:C_0805_2012Metric, symbol Device:C
- removed DI2: Diode_PESD5V0U2BT-Q, Package_TO_SOT_SMD:SOT-23, symbol Personal_Projects:Diode_PESD5V0U2BT-Q
- removed FPC1: FPC_0545481072, Personal_Project:FPC_0545481072, symbol Personal_Projects:FPC_0545481072
- removed FPC2: FPC_ZF5S-20-01-T-WT, Personal_Project:FPC_SAMTEC_ZF5S-20-01-T-WT, symbol Personal_Projects:FPC_ZF5S-20-01-T-WT
- removed FPC4: FPC_0545482072, Personal_Project:FPC_0545482072, symbol Personal_Projects:FPC_0545482072
- removed H5, H6, H7, H8: MountingHole_Pad, MountingHole:MountingHole_3.2mm_M3_Pad, symbol Mechanical:MountingHole_Pad
- removed J10: SPI1_Headers, Connector_PinHeader_2.54mm:PinHeader_2x03_P2.54mm_Horizontal, symbol Connector_Generic:Conn_02x03_Odd_Even
- removed J12: QSPI_Header, Connector_PinHeader_2.54mm:PinHeader_2x05_P2.54mm_Horizontal, symbol Connector_Generic:Conn_02x05_Odd_Even
- removed J13: USR_BTN_EN, Connector_PinHeader_2.54mm:PinHeader_1x02_P2.54mm_Vertical, symbol Connector_Generic:Conn_01x02
- removed J2: I2C1_Headers, Connector_PinHeader_2.54mm:PinHeader_2x03_P2.54mm_Horizontal, symbol Connector_Generic:Conn_02x03_Odd_Even
- removed J4: LPUART1_Headers, Connector_PinHeader_2.54mm:PinHeader_2x03_P2.54mm_Horizontal, symbol Connector_Generic:Conn_02x03_Odd_Even
- removed J5: GPIO_Headder, Connector_PinHeader_2.54mm:PinHeader_2x03_P2.54mm_Horizontal, symbol Connector_Generic:Conn_02x03_Odd_Even
- removed J6: SPI_QSPI_Jumper, Connector_PinHeader_2.54mm:PinHeader_1x03_P2.54mm_Vertical, symbol Connector_Generic:Conn_01x03
- removed MX1: MUX_SN74CB3T3257PWR, Personal_Project:MUX_SN74CB3T3257PWR_SOP65P640X120-16N, symbol Personal_Projects:MUX_SN74CB3T3257PWR
- removed U2: ~, Personal_Project:Button_KMR231GLFS, symbol Personal_Projects:Button_KMR231GLFS
- added DI1: Diode_PESD5V0U2BT-Q, Package_TO_SOT_SMD:SOT-23, symbol Personal_Projects:Diode_PESD5V0U2BT-Q
- added FPC3: FPC_0545482072, Personal_Project:FPC_0545482072, symbol Personal_Projects:FPC_0545482072
- added FPC5: FPC_0545481072, Personal_Project:FPC_0545481072, symbol Personal_Projects:FPC_0545481072
- added J15: I2C1_Headers, Personal_Project:PinHeader_2x03_P2.54mm_Horizontal_Court, symbol Connector_Generic:Conn_02x03_Odd_Even
- added J2: USR_BTN_EN, Connector_PinHeader_2.54mm:PinHeader_1x02_P2.54mm_Vertical, symbol Connector_Generic:Conn_01x02
- added J4: I/O_HDR, Connector_PinHeader_2.54mm:PinHeader_2x04_P2.54mm_Horizontal, symbol Connector_Generic:Conn_02x04_Odd_Even
- added J9: UART1_HDR, Personal_Project:PinHeader_2x03_P2.54mm_Horizontal_Court, symbol Connector_Generic:Conn_02x03_Odd_Even
- added R11, R3: 10k, Resistor_SMD:R_0805_2012Metric, symbol Device:R
- added R2: 33R, Resistor_SMD:R_0805_2012Metric, symbol Device:R
- added U8: ~, Personal_Project:Button_KMR231GLFS, symbol Personal_Projects:Button_KMR231GLFS
- C12: value 100n -> 1uF
- R1: value 33R -> 10k
Connections:
- net GPIO4_FSPIHD_SIO3_R is gone; now on net +3.3V: R1.2
- net +3.3V: now also R11.1, R3.1; no longer C12.1
- net GND: now also C12.1, DI1.3 (CC), FPC3.1, FPC3.10, FPC3.11, FPC3.12, FPC3.14, FPC3.15, FPC3.17, FPC3.18, FPC3.20, FPC3.21 (MP1), FPC3.22 (MP2), FPC3.3, FPC3.4, FPC3.6, FPC3.7, FPC3.9, FPC5.1, FPC5.10, FPC5.11 (MP1), FPC5.12 (MP2), FPC5.3, FPC5.5, FPC5.6, FPC5.8, J15.2 (Pin_2), J15.3 (Pin_3), J15.4 (Pin_4), J15.6 (Pin_6), J4.1 (Pin_1), J4.3 (Pin_3), J4.5 (Pin_5), J4.7 (Pin_7), J9.1 (Pin_1), J9.2 (Pin_2), J9.4 (Pin_4), J9.5 (Pin_5), J9.6 (Pin_6), U8.3, U8.4, U8.5 (GND); no longer C12.2
- net QSPI_CLK: now also FPC3.2
- net QSPI_CS0: now also FPC3.5
- net QSPI_IO0: now also FPC3.8
- net QSPI_IO1: now also FPC3.13
- net QSPI_IO2: now also FPC3.16
- net QSPI_IO3: now also FPC3.19
- net SPI_CLK: now also FPC5.7
- net SPI_CS: now also FPC5.9
- net SPI_MISO: now also FPC5.4
- net SPI_MOSI: now also FPC5.2
- net GPIO4_FSPIHD_SIO3 renamed USR_BTN_P
- net USR_BTN_P: now also C12.2, J2.2 (Pin_2), U8.1, U8.2
- new net: J9.3 (Pin_3), R2.2
- new net I2C_SCL_HDR: DI1.2 (K2), J15.5 (Pin_5), R11.2
- new net I2C_SDA_HDR: DI1.1 (K1), J15.1 (Pin_1), R3.2
- new net I/O_HDR0: J4.2 (Pin_2)
- new net I/O_HDR1: J4.4 (Pin_4)
- new net I/O_HDR2: J4.6 (Pin_6)
- new net I/O_HDR3: J4.8 (Pin_8)
- new net UART1_TX/RX: R2.1
- new net USR_BTN: J2.1 (Pin_1)
Other:
- note added: "Place ESD close to the header"
- note removed: "Chip Select pin on general pin header"
- note removed: "OE control that, when high, disables all switches to their OFF state."
- note removed: "Pin not routed through MUX"
