File: Power_Management.kicad_sch (KiCad schematic)
At the start: 17 parts, among them J7 PWR_SRC_JMP, Q2 MOSFET_SI2333DDS-T1-BE3

Commit message: Update
Parts:
- removed D2: SMAJ6.0A, Personal_Project:DO-214AC-2, symbol Personal_Projects:DIODE_SMAJ6.0A
- removed J7: PWR_SRC_JMP, Connector_PinHeader_2.54mm:PinHeader_1x03_P2.54mm_Vertical, symbol Connector_Generic:Conn_01x03
- removed JST1: JST_S3B-XH-2.54, Personal_Project:JST_S3B-XH-SHDRRA3W64P0X250_1X3_990X1150X610P, symbol Personal_Projects:JST_S3B-XH-A-1_LF_SN
- removed Q2: MOSFET_SI2333DDS-T1-BE3, Personal_Project:MOSFET_ SI2333DDS_SOT_DS-T1-BE3_VIS, symbol Personal_Projects:MOSFET_SI2333DDS-T1-BE3
- removed R3: 100k, Resistor_SMD:R_0805_2012Metric, symbol Device:R
- removed S1: Switch_WS-SLSU SMT Mini Slide, Personal_Project:Switch_WS-SLSU SMT Mini Slide, symbol Personal_Projects:Switch_WS-SLSU SMT Mini Slide
- removed Z2: Diode_BZX84C6V2-7-F, Personal_Project:Diode_BZX84C6V2_SOT96P240X110-3N, symbol Personal_Projects:Diode_BZX84C6V2-7-F
- added D1: SMAJ6.0A, Personal_Project:DO-214AC-2, symbol Personal_Projects:DIODE_SMAJ6.0A
- added J8: PWR_SRC_JMP, Connector_PinHeader_2.54mm:PinHeader_1x03_P2.54mm_Vertical, symbol Connector_Generic:Conn_01x03
- added JST2: JST_S3B-XH-2.54, Personal_Project:JST_S3B-XH-SHDRRA3W64P0X250_1X3_990X1150X610P, symbol Personal_Projects:JST_S3B-XH-A-1_LF_SN
- added Q1: MOSFET_SI2333DDS-T1-BE3, Personal_Project:MOSFET_ SI2333DDS_SOT_DS-T1-BE3_VIS, symbol Personal_Projects:MOSFET_SI2333DDS-T1-BE3
- added R5: 100k, Resistor_SMD:R_0805_2012Metric, symbol Device:R
- added U3: SN74LVC1G07DBVR, Package_TO_SOT_SMD:SOT-23-5, symbol 74xGxx:74LVC1G07
- added Z3: Diode_BZX84C6V2-7-F, Personal_Project:Diode_BZX84C6V2_SOT96P240X110-3N, symbol Personal_Projects:Diode_BZX84C6V2-7-F
Connections:
- net *RST: now also U3.4
- net +3.3V: now also U3.5 (VCC)
- net GND: now also D1.2 (A), JST2.2 (PWR-), R5.2, U3.3 (GND)
- net PWR+: now also JST2.1 (PWR+), Q1.3 (D)
- net PWR+_PS: now reaches C1.1, LDO1.5 (EN), LDO1.8 (IN)
- net PWR+_PS: now also D1.1 (K), J8.1 (Pin_1)
- new net PWR+_GATE: Q1.1 (G), R5.1, Z3.1 (A)
- new net PWR+_PP: J8.2 (Pin_2), Q1.2 (S), Z3.3 (K)
- new net RST_PWR: JST2.3 (RST), U3.2
- new net USB_VBUS+: J8.3 (Pin_3)
- no-connect marks 8 -> 4
Other:
- note removed: "ON/OFF Switch"
- note removed: "Pin 2 connects to one or three"
- moved on the sheet: C1, C10, C11, C4, C6, C8, C9, FB1, LDO1, VS3

Commit message: Update
Parts:
- removed C11, C6: 47u, Capacitor_SMD:C_0805_2012Metric, symbol Device:C_Polarized
- added C6: 100n, Capacitor_SMD:C_0805_2012Metric, symbol Device:C
- C8: value 10n_X7R -> 4u7
- C9: value 10n_X7R -> 100n
- FB1: value BLM21PG601SN1D_0805 -> BLM21AG121BH1D
Connections:
- net +3.3V: now also FB1.2, C6.1; no longer C8.1, FB1.1
- net GND: now also C6.2
- net +3V3A renamed +3.3VA
- net +3.3VA: now also C8.1, FB1.1; no longer FB1.2
Other:
- note added: "120Ohm@100MHz"
- note removed: "To generate 3V3"
- moved on the sheet: C1, C10, C4, LDO1, U3, VS3

Commit message: Update
Parts:
- added H1, H2, H3, H4: MountingHole_Pad, MountingHole:MountingHole_3.2mm_M3_Pad, symbol Mechanical:MountingHole_Pad
- C8: value 4u7 -> 1u
Connections:
- net GND: now also H1.1, H2.1, H3.1, H4.1
- net PWR+_PP: now also J8.1 (Pin_1); no longer J8.2 (Pin_2)
- net PWR+_PS: now also J8.2 (Pin_2); no longer J8.1 (Pin_1)
Other:
- moved on the sheet: J8
