File: ESP32-C6.kicad_sch (KiCad schematic)
At the start: 32 parts, among them U7 ESP32-C6, Y3 ABS07-32.768KHZ-T, Y4 Crystal_ABM8W-40.0000MHZ-4-B1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

Commit message: Update
Parts:
- added J1: Boot_Mode_Control_Pins, Connector_PinHeader_2.54mm:PinHeader_2x03_P2.54mm_Vertical, symbol Connector_Generic:Conn_02x03_Odd_Even
Connections:
- net +3.3V: now also J1.1 (Pin_1), J1.2 (Pin_2)
- net GND: now also J1.5 (Pin_5), J1.6 (Pin_6)
- net GPIO8_BOOT: now also J1.4 (Pin_4)
- net GPIO9_BOOT: now also J1.3 (Pin_3)
- net CHIP_PU_D renamed RST_CHIP_PU_D
Other:
- moved on the sheet: C23, C25, C26, C27, C28, C29, C30, C31, C32, C33, C34, C35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

Commit message: Update
Connections:
- net GPIO20_SDIO_DATA0 renamed GPIO20_FSPICS0
- net GPIO21_SDIO_DATA1 renamed GPIO21_FSPICLK
- net GPIO22_SDIO_DATA2 renamed GPIO22_FSPIQ_MISO/SIO1
- net GPIO23_SDIO_DATA3 renamed GPIO23_FSPID_MOSI/SIO0
Changed lines of the file:
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@@
+		)
+	)
+	(text_box "Notes:\n- The I2C will be set on GPIO10, 11 through the GPIO Matrix\n- QSPI is on GPIO2, 4, 5, 6 ,7 using IO MUX\n- SPI2 to be used must be reprogrammed for "
+		(exclude_from_sim no)
+		(at 19.05 22.225 0)
+		(size 70.485 31.115)
+		(stroke
+			(width 0)
+			(type dash)
+		)
+		(fill
+			(type none)
+		)
+		(effects
+			(font
+				(size 1 1)
+			)
+			(justify left top)
 		)
 	)
@@
 		)
 	)
-	(label "GPIO23_SDIO_DATA3"
+	(label "GPIO23_FSPID_MOSI{slash}SIO0"
 		(at 184.15 53.34 180)
 		(fields_autoplaced yes)
@@
 		)
 	)
-	(label "GPIO22_SDIO_DATA2"
+	(label "GPIO22_FSPIQ_MISO{slash}SIO1"
 		(at 184.15 55.88 180)
 		(fields_autoplaced yes)
@@
 		)
 	)
-	(label "GPIO21_SDIO_DATA1"
+	(label "GPIO21_FSPICLK"
 		(at 184.15 58.42 180)
 		(fields_autoplaced yes)
@@
 		)
 	)
-	(label "GPIO20_SDIO_DATA0"
+	(label "GPIO20_FSPICS0"
 		(at 184.15 60.96 180)
 		(fields_autoplaced yes)
@@
 		)
 	)
-	(hierarchical_label "GPIO23_SDIO_DATA3"
+	(hierarchical_label "GPIO23_FSPID_MOSI{slash}SIO0"
 		(shape bidirectional)
 		(at 184.15 53.34 0)
@@
 		)
 	)
-	(hierarchical_label "GPIO20_SDIO_DATA0"
+	(hierarchical_label "GPIO20_FSPICS0"
 		(shape bidirectional)
 		(at 184.15 60.96 0)
@@
 		)
 	)
-	(hierarchical_label "GPIO22_SDIO_DATA2"
+	(hierarchical_label "GPIO22_FSPIQ_MISO{slash}SIO1"
 		(shape bidirectional)
 		(at 184.15 55.88 0)
@@
 		)
 	)
-	(hierarchical_label "GPIO21_SDIO_DATA1"
+	(hierarchical_label "GPIO21_FSPICLK"
 		(shape bidirectional)
 		(at 184.15 58.42 0)

Commit message: Update
Parts:
- removed C26: 10u, Capacitor_SMD:C_0805_2012Metric, symbol Device:C
- removed C27: 1u, Capacitor_SMD:C_0805_2012Metric, symbol Device:C
- removed C28: 100n, Capacitor_SMD:C_0805_2012Metric, symbol Device:C
- removed C7: 1uF, Capacitor_SMD:C_0805_2012Metric, symbol Device:C
- removed L2: 2n, Inductor_SMD:L_0805_2012Metric_Pad1.05x1.20mm_HandSolder, symbol Device:L
- removed U6: ~, Personal_Project:Button_KMR231GLFS, symbol Personal_Projects:Button_KMR231GLFS
- R8: value 10k -> 33R
Connections:
- net +3.3V: no longer C29.1, C31.1, R8.2, U7.37 (VDDA1), U7.40 (VDDA2)
- net GPIO4_FSPIHD_SIO3: now also R8.1; no longer U7.10 (MTMS)
- net RST_CHIP_PU_D: no longer R8.1
- net XTAL_32K_P: now reaches C23.1, R9.2, U7.6 (XTAL_32K_P), Y3.1
- net XTAL_32K_N: now reaches C25.1, R9.1, U7.7 (XTAL_32K_N), Y3.2
- net +3.3VA: now reaches C30.1, U7.2 (VDDA3P3_1), U7.3 (VDDA3P3_2)
- net +3.3VA: now also C29.1, C31.1, U7.37 (VDDA1), U7.40 (VDDA2)
- new net GPIO4_FSPIHD_SIO3_R: R8.2, U7.10 (MTMS)
Other:
- note added: "CHIP_PU pin can enable the chip when it is high and reset the chip when it is low"
- note removed: "From manual (delay circuit)"
- moved on the sheet: C30, R19, R21, R22

Commit message: Update
Changed lines of the file:
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@@
 	(label "XTAL_32K_N"
 		(at 110.49 107.95 0)
+		(fields_autoplaced yes)
 		(effects
 			(font
@@
 	(label "XTAL_32K_P"
 		(at 110.49 105.41 0)
+		(fields_autoplaced yes)
 		(effects
 			(font
@@
 		(dnp no)
 		(property "Reference" "C23"
-			(at 61.468 106.934 90)
-			(effects
-				(font
+			(at 60.706 106.934 90)
+			(effects
+				(font
