File: ESP32C6_Board.kicad_sch (KiCad schematic)
At the start: 72 parts, among them J1 SDIO_Header, J10 JST_XH_2.54_Plug, J11 SPI_QSPI_Jumper, J16 Power_Selector_Jumper, J18 USR_BTN_EN, J19 SPI1_Headers, J2 USB_B_Micro, J3 Boot_Mode_Control_Pins, J5 3V_Selection_Header, J6 LPUART1_Headers, J7 I2C1_Headers, J8 GPIO_Headder, J9 QSPI_Header, Q1 MOSFET_SI2333DDS-T1-BE3, U1 ESP32-C6, U2 W25Q128JVSQ_SOIC208-mil, U3 USBLC6-2SC6, Y1 Crystal_ABM8W-40.0000MHZ-4-B1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, Y2 ABS07-32.768KHZ-T

Commit message: Update
Parts:
- removed J1: SDIO_Header, Connector_PinHeader_2.54mm:PinHeader_2x06_P2.54mm_Horizontal, symbol Connector_Generic:Conn_02x06_Odd_Even
- added FPC1, FPC2: FPC_ZF5S-20-01-T-WT, Personal_Project:FPC_SAMTEC_ZF5S-20-01-T-WT, symbol Personal_Projects:FPC_ZF5S-20-01-T-WT
Connections:
- net GND: now also J8.3 (Pin_3), FPC1.01, FPC1.03, FPC1.04, FPC1.06, FPC1.07, FPC1.09, FPC1.10, FPC1.12, FPC1.13, FPC1.15, FPC1.16, FPC1.18, FPC1.19, FPC2.01, FPC2.03, FPC2.04, FPC2.06, FPC2.07, FPC2.09, FPC2.10, FPC2.12, FPC2.13, FPC2.15, FPC2.16, FPC2.18, FPC2.19
- net GPIO18_SDIO_CMD: now also FPC1.17, FPC2.17
- net GPIO19_SDIO_CLK: now also FPC1.14, FPC2.14
- net GPIO20_SDIO_DATA0: now also FPC1.11, FPC2.11
- net GPIO21_SDIO_DATA1: now also FPC1.08, FPC2.08
- net GPIO22_SDIO_DATA2: now also FPC1.05, FPC2.05
- net GPIO23_SDIO_DATA3: now also FPC1.02, FPC2.02
- net GPIO15 renamed GPIO15_SDIO_INT
- net GPIO15_SDIO_INT: now also FPC1.20, FPC2.20; no longer J8.3 (Pin_3)
Other:
- moved on the sheet: J6, J7, J8

Commit message: Update
Parts:
- removed C1, C4, C9: 1u, Capacitor_SMD:C_0805_2012Metric, symbol Device:C
- removed C10, C11, C12, C5, C6: 100n, Capacitor_SMD:C_0805_2012Metric, symbol Device:C
- removed C13, C14: 2p, Capacitor_SMD:C_0805_2012Metric, symbol Device:C
- removed C17, C8: 15p, Capacitor_SMD:C_0805_2012Metric, symbol Device:C
- removed C2: 10n, Capacitor_SMD:C_0805_2012Metric, symbol Device:C
- removed C21: 1uF, Capacitor_SMD:C_0805_2012Metric, symbol Device:C
- removed C3: 10u, Capacitor_SMD:C_0805_2012Metric, symbol Device:C
- removed FPC2: FPC_ZF5S-20-01-T-WT, Personal_Project:FPC_SAMTEC_ZF5S-20-01-T-WT, symbol Personal_Projects:FPC_ZF5S-20-01-T-WT
- removed L1: 2n, Inductor_SMD:L_0805_2012Metric_Pad1.05x1.20mm_HandSolder, symbol Device:L
- removed R11, R12, R13, R14, R15, R5: 0R, Resistor_SMD:R_0805_2012Metric, symbol Device:R
- removed R17, R18, R4, R7: 33R, Resistor_SMD:R_0805_2012Metric, symbol Device:R
- removed R20: 10k, Resistor_SMD:R_0805_2012Metric, symbol Device:R
- removed R3: 100k, Resistor_SMD:R_0805_2012Metric, symbol Device:R
- removed U1: ESP32-C6, Personal_Project:ESP32C6_QFN40P500X500X90-41N-D, symbol Personal_Projects:ESP32-C6
- removed U5: ~, Personal_Project:Button_KMR231GLFS, symbol Personal_Projects:Button_KMR231GLFS
- removed Y1: Crystal_ABM8W-40.0000MHZ-4-B1U-T3, Personal_Project:CRYSTAL4_ABM10W-40.0000MHZ-8-B1U-T3_ABR, symbol Personal_Projects:Crystal_ABM10W-40.0000MHZ-8-B1U-T3
- removed Y2: ABS07-32.768KHZ-T, Personal_Project:Crystal_ABS07, symbol Device:Crystal_Small
- added DI1: Diode_PESD5V0U2BT-Q, Package_TO_SOT_SMD:SOT-23, symbol Personal_Projects:Diode_PESD5V0U2BT-Q
Connections:
- net GND: now also DI1.3 (CC)
- net GPIO10_I2C_SCL: now also DI1.1 (K1)
- net GPIO11_I2C_SDA: now also DI1.2 (K2)
Other:
- added sheet ESP32-C6 (ESP32-C6.kicad_sch)
- note removed: "Boot Mode Control GPIO8 and 9"
- note removed: "FSPICLK - CLK"
- note removed: "FSPID - MISO"
- note removed: "FSPIHD - HOLD"
- note removed: "FSPIQ - MOSI"
- note removed: "FSPIWP - Write Protect"
- note removed: "From manual (delay circuit)"
- note removed: "Pin VDD_SPI can serve as the power supply for the external device at 3.3 V (typical value), provided by VDDPST2 via RSPI."
- note removed: "Placeholder Resistors"
- note removed: "Resistor is optional (5 MΩ < R ≤ 10 MΩ)"
- note removed: "UART0 interface"
- note removed: "pg797 Technical: Signals Used in Various SPI Modes"
- moved on the sheet: J19, J6, J7, J8, J9, R6

Commit message: Update
Parts:
- removed ANT1: Antenna_2450AT18D0100001E, Personal_Project:Antenna_2450AT18D0100001E, symbol Personal_Projects:Antenna_2450AT18D0100001E
- removed C15, C16: 100n, Capacitor_SMD:C_0603_1608Metric, symbol Device:C
- removed C18, C19: 1u, Capacitor_SMD:C_0805_2012Metric, symbol Device:C
- removed C20: 1uF, Capacitor_SMD:C_0805_2012Metric, symbol Device:C
- removed C22: 4u7, Capacitor_SMD:C_0805_2012Metric, symbol Device:C
- removed C24: 100n, Capacitor_SMD:C_0805_2012Metric, symbol Device:C
- removed D1: ESD_TSD03DYFR, Personal_Project:ESD_TSD05DYFR_SOD2613X100N, symbol Personal_Projects:ESD_TSD05DYFR
- removed D3: ESD_TSD05DYFR, Personal_Project:ESD_TSD05DYFR_SOD2613X100N, symbol Personal_Projects:ESD_TSD05DYFR
- removed DI1: Diode_PESD5V0U2BT-Q, Package_TO_SOT_SMD:SOT-23, symbol Personal_Projects:Diode_PESD5V0U2BT-Q
- removed FPC1: FPC_ZF5S-20-01-T-WT, Personal_Project:FPC_SAMTEC_ZF5S-20-01-T-WT, symbol Personal_Projects:FPC_ZF5S-20-01-T-WT
- removed H1, H2, H3, H4: MountingHole_Pad, MountingHole:MountingHole_3.2mm_M3_Pad, symbol Mechanical:MountingHole_Pad
- removed J10: JST_XH_2.54_Plug, Personal_Project:Connector_Power2pin_SHDRRA2W80P0X250_1X2_740X1150X610P, symbol Personal_Projects:Connector_Power2pin_JST_XH_2.54_Plug
- removed J11: SPI_QSPI_Jumper, Connector_PinHeader_2.54mm:PinHeader_1x03_P2.54mm_Vertical, symbol Connector_Generic:Conn_01x03
- removed J16: Power_Selector_Jumper, Connector_PinHeader_2.54mm:PinHeader_2x03_P2.54mm_Vertical, symbol Connector_Generic:Conn_02x03_Odd_Even
- removed J18: USR_BTN_EN, Connector_PinHeader_2.54mm:PinHeader_1x02_P2.54mm_Vertical, symbol Connector_Generic:Conn_01x02
- removed J19: SPI1_Headers, Connector_PinHeader_2.54mm:PinHeader_2x03_P2.54mm_Horizontal, symbol Connector_Generic:Conn_02x03_Odd_Even
- removed J2: USB_B_Micro, Connector_USB:USB_Micro-B_Molex-105017-0001, symbol Connector:USB_B_Micro
- removed J3: Boot_Mode_Control_Pins, Connector_PinHeader_2.54mm:PinHeader_2x03_P2.54mm_Vertical, symbol Connector_Generic:Conn_02x03_Odd_Even
- removed J5: 3V_Selection_Header, Connector_PinHeader_2.54mm:PinHeader_1x03_P2.54mm_Vertical, symbol Connector_Generic:Conn_01x03
- removed J6: LPUART1_Headers, Connector_PinHeader_2.54mm:PinHeader_2x03_P2.54mm_Horizontal, symbol Connector_Generic:Conn_02x03_Odd_Even
- removed J7: I2C1_Headers, Connector_PinHeader_2.54mm:PinHeader_2x03_P2.54mm_Horizontal, symbol Connector_Generic:Conn_02x03_Odd_Even
- removed J8: GPIO_Headder, Connector_PinHeader_2.54mm:PinHeader_2x03_P2.54mm_Horizontal, symbol Connector_Generic:Conn_02x03_Odd_Even
- removed J9: QSPI_Header, Connector_PinHeader_2.54mm:PinHeader_2x05_P2.54mm_Horizontal, symbol Connector_Generic:Conn_02x05_Odd_Even
- removed L3: 2n, Inductor_SMD:L_0603_1608Metric, symbol Device:L
- removed LDO1: LDO_TLV75733PDBVR, Personal_Project:LDO_SOT95P280X145-5N, symbol Personal_Projects:LDO_TLV75733PDBVR
- removed MX3: MUX_SN74CB3T3257PWR, Personal_Project:MUX_SN74CB3T3257PWR_SOP65P640X120-16N, symbol Personal_Projects:MUX_SN74CB3T3257PWR
- removed Q1: MOSFET_SI2333DDS-T1-BE3, Personal_Project:MOSFET_ SI2333DDS_SOT_DS-T1-BE3_VIS, symbol Personal_Projects:MOSFET_SI2333DDS-T1-BE3
- removed R1, R16, R2: 100k, Resistor_SMD:R_0805_2012Metric, symbol Device:R
- removed R6: 33R, Resistor_SMD:R_0805_2012Metric, symbol Device:R
- removed S2: Switch_WS-SLSU SMT Mini Slide, Personal_Project:Switch_WS-SLSU SMT Mini Slide, symbol Personal_Projects:Switch_WS-SLSU SMT Mini Slide
- removed U2: W25Q128JVSQ_SOIC208-mil, Package_SO:SOIC-8_5.23x5.23mm_P1.27mm, symbol Memory_Flash:W25Q128JVS
- removed U3: USBLC6-2SC6, Package_TO_SOT_SMD:SOT-23-6, symbol Power_Protection:USBLC6-2SC6
- removed U4: ~, Personal_Project:Button_KMR231GLFS, symbol Personal_Projects:Button_KMR231GLFS
- removed Z1: Diode_BZX84C6V2-7-F, Personal_Project:Diode_BZX84C6V2_SOT96P240X110-3N, symbol Personal_Projects:Diode_BZX84C6V2-7-F
Connections:
- no-connect marks 5 -> 0
Other:
- added sheet Interfaces (Interfaces.kicad_sch)
- added sheet Power_Management (Power_Management.kicad_sch)
- added sheet RF_USB_Memory (RF_USB_Memory.kicad_sch)
- sheet ESP32-C6 ports: added GPIO15_SDIO_INT, RST_CHIP_PU_D; removed GPIO8_BOOT, GPIO9_BOOT
- note removed: "-----Impedance Matching Look for high Q capacitors (more ideal)"
- note removed: "5.5V Max Voltage of the LDO"
- note removed: "Chip Select pin on general pin header"
- note removed: "Fixed Output"
- note removed: "If shutdown capability is not required, connect EN to IN."
- note removed: "Input voltage range: 1.45V to 5.5V"
- note removed: "Input voltage range: 1.45V to 5.5V Abs Max Vin is 6V"
- note removed: "LDO Input voltage range: 1.45V to 5.5V Abs Max Vin is 6V"
- note removed: "OE control that, when high, disables all switches to their OFF state."
- note removed: "ON/OFF Switch"
- note removed: "Overvoltage protection for the PMOSFET VGS (VGS max is 8V)"
- note removed: "Pin not routed through MUX"
- note removed: "Polarity Protection"

Commit message: Update
Other:
- sheet RF_USB_Memory ports: added USB_D2+_DI, USB_D2-_DI; removed USB_D+, USB_D-
Changed lines of the file:
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@@
+	(wire
+		(pts
+			(xy 92.71 76.2) (xy 116.84 76.2)
+		)
+		(stroke
+			(width 0)
+			(type default)
+		)
+	)
 	(wire
 		(pts
@@
 	(wire
 		(pts
+			(xy 173.99 53.34) (xy 198.12 53.34)
+		)
+		(stroke
+			(width 0)
+			(type default)
+		)
+	)
+	(wire
+		(pts
 			(xy 92.71 78.74) (xy 116.84 78.74)
 		)
@@
 	(wire
 		(pts
-			(xy 173.99 53.34) (xy 198.12 53.34)
-		)
-		(stroke
-			(width 0)
-			(type default)
-		)
-	)
-	(wire
-		(pts
 			(xy 173.99 58.42) (xy 198.12 58.42)
 		)
@@
 		(pts
 			(xy 92.71 43.18) (xy 116.84 43.18)
-		)
-		(stroke
-			(width 0)
-			(type default)
-		)
-	)
-	(wire
-		(pts
-			(xy 92.71 76.2) (xy 116.84 76.2)
 		)
 		(stroke
@@
 			)
 		)
-		(pin "USB_D-" bidirectional
-			(at 92.71 78.74 0)
-			(effects
-				(font
-					(size 1.27 1.27)
-				)
-				(justify right)
-			)
-		)
-		(pin "USB_D+" bidirectional
-			(at 92.71 76.2 0)
-			(effects
-				(font
-					(size 1.27 1.27)
-				)
-				(justify right)
-			)
-		)
 		(pin "SPICS0_Chip_Select" bidirectional
 			(at 92.71 48.26 0)
@@
 			(effects
 				(font
+					(size 1.27 1.27)
+				)
+				(justify right)
+			)
+		)
+		(pin "USB_D2+_DI" bidirectional
+			(at 92.71 76.2 0)
+			(effects
+				(font
+					(size 1.27 1.27)
+				)
+				(justify right)
+			)
+		)
+		(pin "USB_D2-_DI" bidirectional
+			(at 92.71 78.74 0)
+			(effects
+				(font

Commit message: Update
Other:
- sheet ESP32-C6 ports: added GPIO20_FSPICS0, GPIO21_FSPICLK, GPIO22_FSPIQ_MISO/SIO1, GPIO23_FSPID_MOSI/SIO0; removed GPIO20_SDIO_DATA0, GPIO21_SDIO_DATA1, GPIO22_SDIO_DATA2, GPIO23_SDIO_DATA3
- sheet Interfaces ports: added I2C_SCL_HDR, I2C_SDA_HDR, I/O_HDR0, I/O_HDR1, I/O_HDR2, I/O_HDR3, QSPI_CLK, QSPI_CS0, QSPI_IO0, QSPI_IO1, QSPI_IO2, QSPI_IO3, SPI_CLK, SPI_CS, SPI_MISO, SPI_MOSI, UART1_TX/RX, USR_BTN; removed GPIO10_I2C_SCL, GPIO11_I2C_SDA, GPIO15_SDIO_INT, GPIO16_U0RXD, GPIO17_U0TXD, GPIO18_SDIO_CMD, GPIO19_SDIO_CLK, GPIO20_SDIO_DATA0, GPIO21_SDIO_DATA1, GPIO22_SDIO_DATA2, GPIO23_SDIO_DATA3

Commit message: Update
Other:
- added sheet Camera (Camera.kicad_sch)
- added sheet LCD (LCD_Camera.kicad_sch)
Changed lines of the file:
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@@
+	)
+	(sheet
+		(at 45.72 168.91)
+		(size 45.085 19.685)
+		(fields_autoplaced yes)
+		(stroke
+			(width 0.1524)
+			(type solid)
+		)
+		(fill
+			(color 0 255 255 1.0000)
+		)
+		(property "Sheetname" "LCD"
+			(at 45.72 168.1984 0)
+			(effects
+				(font
+					(size 1.27 1.27)
+				)
+				(justify left bottom)
+			)
+		)
+		(property "Sheetfile" "LCD_Camera.kicad_sch"
+			(at 45.72 189.1796 0)
+			(effects
+				(font
+					(size 1.27 1.27)
+				)
+				(justify left top)
+			)
+		)
+		(instances
+			(project "ESP32C6_Board"
+				(path "/beafeceb-d7f8-4966-bdc7-36ccea772b2f"
+					(page "6")
+				)
+			)
+		)
+	)
+	(sheet
+		(at 120.65 135.255)
+		(size 45.085 18.415)
+		(fields_autoplaced yes)
+		(stroke
+			(width 0.1524)
+			(type solid)
+		)
+		(fill
+			(color 0 255 255 1.0000)
+		)
+		(property "Sheetname" "Camera"
+			(at 120.65 134.5434 0)
+			(effects
+				(font
+					(size 1.27 1.27)
+				)
+				(justify left bottom)
+			)
+		)
+		(property "Sheetfile" "Camera.kicad_sch"
+			(at 120.65 154.2546 0)
+			(effects
+				(font
+					(size 1.27 1.27)
+				)
+				(justify left top)
+			)
+		)
+		(instances
+			(project "ESP32C6_Board"
+				(path "/beafeceb-d7f8-4966-bdc7-36ccea772b2f"
+					(page "7")
+				)
+			)
+		)
 	)
 	(sheet

Commit message: Update
Other:
- added sheet ESP32-S3 (ESP32-S3.kicad_sch)
Changed lines of the file:
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@@
+	)
+	(sheet
+		(at 120.65 163.195)
+		(size 45.085 16.51)
+		(fields_autoplaced yes)
+		(stroke
+			(width 0.1524)
+			(type solid)
+		)
+		(fill
+			(color 0 255 255 1.0000)
+		)
+		(property "Sheetname" "ESP32-S3"
+			(at 120.65 162.4834 0)
+			(effects
+				(font
+					(size 1.27 1.27)
+				)
+				(justify left bottom)
+			)
+		)
+		(property "Sheetfile" "ESP32-S3.kicad_sch"
+			(at 120.65 180.2896 0)
+			(effects
+				(font
+					(size 1.27 1.27)
+				)
+				(justify left top)
+			)
+		)
+		(instances
+			(project "ESP32C6_Board"
+				(path "/beafeceb-d7f8-4966-bdc7-36ccea772b2f"
+					(page "8")
+				)
+			)
+		)
 	)
 	(sheet
