File: ESP32-S3.kicad_sch (KiCad schematic)
At the start: 4 parts, among them Y1 Crystal_ABM8W-40.0000MHZ-4-B1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

Commit message: Update
Parts:
- added C28, C41, C46: 1u, Capacitor_SMD:C_0805_2012Metric, symbol Device:C
- added C38: 10n, Capacitor_SMD:C_0805_2012Metric, symbol Device:C
- added C39, C42, C43, C44, C45: 100n, Capacitor_SMD:C_0805_2012Metric, symbol Device:C
- added C40: 10u, Capacitor_SMD:C_0805_2012Metric, symbol Device:C
- added L3: 2n, Inductor_SMD:L_1008_2520Metric, symbol Device:L
- added L4: 25n, Inductor_SMD:L_1008_2520Metric, symbol Device:L
- added R15: 100k, Resistor_SMD:R_0805_2012Metric, symbol Device:R
- added U1: W25Q128JVSQ_SOIC208-mil, Package_SO:SOIC-8_5.23x5.23mm_P1.27mm, symbol Memory_Flash:W25Q128JVS
Connections:
- net GND: now also MCU1.57 (GND), C28.2, C38.2, C39.2, C40.2, C41.2, C42.2, C43.2, C44.2, C45.2, C46.2, U1.4 (GND)
- net at C26.1, Y1.1: now also L4.1; no longer MCU1.21 (XTAL_32K_P)
- net at C27.1, Y1.3: now also MCU1.53 (XTAL_N); no longer MCU1.22 (XTAL_32K_N)
- net GPIO5: now reaches MCU1.10 (GPIO5)
- net GPIO6: now reaches MCU1.11 (GPIO6)
- net GPIO7: now reaches MCU1.12 (GPIO7)
- net GPIO8: now reaches MCU1.13 (GPIO8)
- net GPIO9: now reaches MCU1.14 (GPIO9)
- net GPIO10: now reaches MCU1.15 (GPIO10)
- net GPIO11: now reaches MCU1.16 (GPIO11)
- net GPIO12: now reaches MCU1.17 (GPIO12)
- net GPIO13: now reaches MCU1.18 (GPIO13)
- net GPIO14: now reaches MCU1.19 (GPIO14)
- net at MCU1.2 (VDD3P3): now also MCU1.3 (VDD3P3__1), C42.1, L3.1
- net +3.3V: now reaches MCU1.20 (VDD3P3_RTC)
- net +3.3V: now also MCU1.46 (VDD3P3_CPU), MCU1.55 (VDDA1), MCU1.56 (VDDA2), C28.1, C38.1, C39.1, C40.1, C41.1, C43.1, C44.1, L3.2
- net GPIO17: now reaches MCU1.23 (GPIO17)
- net GPIO18: now reaches MCU1.24 (GPIO18)
- net GPIO19: now reaches MCU1.25 (GPIO19)
- net GPIO20: now reaches MCU1.26 (GPIO20)
- net GPIO21: now reaches MCU1.27 (GPIO21)
- net SPICS1: now reaches MCU1.28 (SPICS1)
- net VDDSPI+: now reaches MCU1.29 (VDD_SPI)
- net VDDSPI+: now also C45.1, C46.1
- net SPIHD: now reaches MCU1.30 (SPIHD)
- net SPIWP: now reaches MCU1.31 (SPIWP)
- net SPICS0: now reaches MCU1.32 (SPICS0)
- net SPICLK: now reaches MCU1.33 (SPICLK)
- net SPIQ: now reaches MCU1.34 (SPIQ)
- net SPID: now reaches MCU1.35 (SPID)
- net SPICLK_N: now reaches MCU1.36 (SPICLK_N)
- net SPICLK_P: now reaches MCU1.37 (SPICLK_P)
- net GPIO33: now reaches MCU1.38 (GPIO33)
- net GPIO34: now reaches MCU1.39 (GPIO34)
- net CHIP_PU: now reaches MCU1.4 (CHIP_PU)
- net GPIO35: now reaches MCU1.40 (GPIO35)
- net GPIO36: now reaches MCU1.41 (GPIO36)
- net GPIO37: now reaches MCU1.42 (GPIO37)
- net GPIO38: now reaches MCU1.43 (GPIO38)
- net MTCK: now reaches MCU1.44 (MTCK)
- net MTDO: now reaches MCU1.45 (MTDO)
- net MTDI: now reaches MCU1.47 (MTDI)
- net MTMS: now reaches MCU1.48 (MTMS)
- net U0TXD: now reaches MCU1.49 (U0TXD)
- net GPIO0: now reaches MCU1.5 (GPIO0)
- net U0RXD: now reaches MCU1.50 (U0RXD)
- net GPIO45: now reaches MCU1.51 (GPIO45)
- net GPIO46: now reaches MCU1.52 (GPIO46)
- net at MCU1.54 (XTAL_P): now also L4.2
- net GPIO1: now reaches MCU1.6 (GPIO1)
- net GPIO2: now reaches MCU1.7 (GPIO2)
- net GPIO3: now reaches MCU1.8 (GPIO3)
- net GPIO4: now reaches MCU1.9 (GPIO4)
- new net +3.3V_VDD_SPI: R15.1, U1.8 (VCC)
- new net GPIO15: MCU1.21 (XTAL_32K_P)
- new net GPIO16: MCU1.22 (XTAL_32K_N)
- new net SPICLK_Clock: U1.6 (CLK)
- new net SPICS0_Chip_Select: R15.2, U1.1 (~{CS})
- new net SPID_Data_In: U1.5 (DI(IO0))
- new net SPIHD_Hold: U1.7 (IO3)
- new net SPIQ_Data_Out: U1.2 (DO(IO1))
- new net SPIWP_Write_Protect: U1.3 (IO2)
- no-connect marks 0 -> 1
Other:
- note added: "The value of L4 varies with the actual PCB board. R4 could be a resistor or inductor, the initial value is suggested to be 24 nH."
- moved on the sheet: C26, C27, MCU1, Y1
